File: hardware/NS FPGA.kicad_pcb (KiCad board)
At the start: 6 copper layers, 27.2 x 64.8 mm, 46 parts, among them J1 USB_C_Receptacle_USB2.0_14P, J2 Conn_01x24_Pin, J3 Conn_01x24_Pin, J4 Jtag PIN, Q1 BSS138, SW1 SW_Push, U2 CP2102N-Axx-xQFN24, U3 AP2112K-3.3, U4 AP2112K-1.2, Y1 SG-8002CE(24.0000M)

Commit message: Complete PCB layout, add documentation image, and update README
Parts:
- added G***: LOGO, LOGO, F.Cu at (100.1, 121.0)
Connections:
- J2 pad 21: /IO_B4 -> unconnected-(J2-Pin_21-Pad21)
- J2 pad 23: /IO_B5 -> +3V3
- J2 pad 24: /IO_B6 -> GND
Routing:
- net +3V3: track 31.8 -> 142.7 mm, vias 8 -> 14
- net +5V: track 0.00 -> 87.2 mm, vias 0 -> 2
- net GND: track 0.71 -> 37.5 mm, vias 0 -> 9
- net +1V2: track 6.40 -> 35.0 mm, vias 3 -> 6
- net /IO_G5: track 12.8 -> 19.2 mm
- net Net-(U2-~{RST}): track 7.95 -> 3.35 mm, vias 0 -> 2
- net Net-(U2-VDD): track 2.99 -> 5.77 mm
- net Net-(D1-A): track 0.00 -> 1.28 mm
- net /IO_C8: track 29.3 -> 30.6 mm
- added copper zone on In3.Cu, net +1V2
- added copper zone on In3.Cu, net +5V
- added copper zone on F.Cu, net GND
- added copper zone on In1.Cu, net GND
- added copper zone on In4.Cu, net GND
Other:
- board text added: "Designed by: Muhammad Uzzam Butt"
- board text added: "Designed in Pakistan"
- board text added: "N | NorthernStudios"
- board text added: "northernstudios.cc"

Commit message: added pin numbering silkscreen
Connections:
- J2 pad 2: /IO_D6 -> unconnected-(J2-Pin_2-Pad2)
Other:
- board text added: "3V3"
- board text added: "5V"
- board text added: "A1"
- board text added: "A2"
- board text added: "A3"
- board text added: "A4"
- board text added: "A5"
- board text added: "A6"
- board text added: "B1"
- board text added: "B2"
- board text added: "B3"
- board text added: "C2"
- board text added: "C4"
- board text added: "C5"
- board text added: "C7"
- board text added: "C8"
- board text added: "D1"
- board text added: "D7"
- board text added: "D8"
- board text added: "E1"
- board text added: "E8"
- board text added: "F1"
- board text added: "G3"
- board text added: "G4"
- board text added: "G5"
- board text added: "GND"
- board text added: "H2"
- board text added: "H3"
- board text added: "H4"
- board text added: "H5"
- board text added: "H6"
- board text added: "H7"
- board text added: "H8"
- board text added: "TCK"
- board text added: "TDI"
- board text added: "TDO"
- board text added: "TMS"
