File: hardware/NS FPGA.kicad_sch (KiCad schematic)
At the start: 46 parts, among them J1 USB_C_Receptacle_USB2.0_14P, J2 Conn_01x24_Pin, J3 Conn_01x24_Pin, J4 Jtag PIN, Q1 BSS138, SW1 SW_Push, U2 CP2102N-Axx-xQFN24, U3 AP2112K-3.3, U4 AP2112K-1.2, Y1 SG-8002CE(24.0000M)

Commit message: Complete PCB layout, add documentation image, and update README
Connections:
- net +3V3: now also J2.23 (Pin_23)
- net GND: now also J2.24 (Pin_24)
- net IO_B4: no longer J2.21 (Pin_21)
- net IO_B5: no longer J2.23 (Pin_23)
- net IO_B6: no longer J2.24 (Pin_24)
- no-connect marks 25 -> 31
Changed lines of the file:
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@@
-		)
-	)
-	(text_box "Header Pins"
-		(exclude_from_sim no)
-		(at 196.85 144.78 0)
-		(size 69.85 124.46)
-		(margins 0.9525 0.9525 0.9525 0.9525)
-		(stroke
-			(width 0)
-			(type solid)
-		)
-		(fill
-			(type none)
-		)
-		(effects
-			(font
-				(size 2.54 2.54)
-			)
-			(justify left top)
 		)
 	)
@@
 	)
 	(junction
+		(at 209.55 161.29)
+		(diameter 0)
+		(color 0 0 0 0)
+	)
+	(junction
 		(at 246.38 81.28)
 		(diameter 0)
@@
 	)
 	(no_connect
+		(at 125.73 190.5)
+	)
+	(no_connect
+		(at 243.84 186.69)
+	)
+	(no_connect
 		(at 326.39 105.41)
 	)
@@
 	)
 	(no_connect
+		(at 243.84 189.23)
+	)
+	(no_connect
 		(at 326.39 85.09)
 	)
 	(no_connect
+		(at 121.92 190.5)
+	)
+	(no_connect
 		(at 326.39 87.63)
 	)
@@
 	)
 	(no_connect
+		(at 129.54 190.5)
+	)
+	(no_connect
 		(at 326.39 102.87)
 	)
@@
 	)
 	(no_connect
+		(at 219.71 166.37)
+	)
+	(no_connect
 		(at 99.06 255.27)
 	)
@@
 	(wire
 		(pts
-			(xy 209.55 176.53) (xy 209.55 158.75)
+			(xy 209.55 176.53) (xy 209.55 161.29)
 		)
 		(stroke
@@
 	(wire
 		(pts
+			(xy 209.55 161.29) (xy 209.55 158.75)
+		)
+		(stroke
+			(width 0)
+			(type default)
+		)
+	)
+	(wire
+		(pts
 			(xy 332.74 168.91) (xy 332.74 171.45)
 		)
@@
 	(wire
 		(pts
+			(xy 231.14 158.75) (xy 231.14 163.83)
+		)
+		(stroke
+			(width 0)
+			(type default)
+		)
+	)
+	(wire
+		(pts
 			(xy 219.71 212.09) (xy 231.14 212.09)
 		)
@@
 	(wire
 		(pts
+			(xy 209.55 161.29) (xy 219.71 161.29)
+		)
+		(stroke
+			(width 0)
+			(type default)
+		)
+	)
+	(wire
+		(pts
 			(xy 331.47 229.87) (xy 331.47 231.14)
 		)
@@
 		(pts
 			(xy 372.11 87.63) (xy 372.11 88.9)
+		)
+		(stroke
+			(width 0)
+			(type default)
+		)
+	)
+	(wire
+		(pts
+			(xy 219.71 158.75) (xy 231.14 158.75)
 		)
 		(stroke
@@
 		)
 	)
-	(label "IO_B4"
-		(at 219.71 166.37 180)
-		(effects
-			(font
-				(size 1.27 1.27)
-				(thickness 0.254)
-				(bold yes)
-				(italic yes)
-			)
-			(justify right bottom)
-		)
-	)
 	(label "IO_G3"
 		(at 87.63 255.27 270)
@@
 		)
 	)
-	(label "IO_B6"
-		(at 219.71 158.75 180)
-		(effects
-			(font
-				(size 1.27 1.27)
-				(thickness 0.254)
-				(bold yes)
-				(italic yes)
-			)
-			(justify right bottom)
-		)
-	)
 	(label "JTAG_TMS"
 		(at 92.71 124.46 180)
@@
 		(effects
 			(font
-				(size 1.27 1.27)
-				(thickness 0.254)
-				(bold yes)
-				(italic yes)
-			)
-			(justify right bottom)
-		)
-	)
-	(label "IO_B5"
-		(at 219.71 161.29 180)
-		(effects
-			(font

Commit message: added pin numbering silkscreen
Connections:
- net IO_D6: no longer names the net of J2.2 (Pin_2)
- no-connect marks 31 -> 32
Changed lines of the file:
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@@
+	)
+	(no_connect
+		(at 219.71 214.63)
 	)
 	(no_connect
@@
 		)
 	)
-	(label "IO_D6"
-		(at 219.71 214.63 180)
-		(effects
-			(font
-				(size 1.27 1.27)
-				(thickness 0.254)
-				(bold yes)
-				(italic yes)
-			)
-			(justify right bottom)
-		)
-	)
